Commit message: Recover the car

File: cam/urdf/gazebo_robot.urdf.xacro (robot description, xacro)
@@ -3,5 +3,5 @@
 	<xacro:include filename="$(find cam)/urdf/gazebo_robot.xacro" />
 	<xacro:include filename="$(find cam)/urdf/camera.xacro" />
-	<xacro:property name="camera_offset_z" value="0.035" />
+	<xacro:property name="camera_offset_z" value="0.85" />
 	<!-- Body of robot, with plates, standoffs and Create (including sim sensors) -->
 	<robot_body/>
@@ -14,5 +14,5 @@
 	<xacro:usb_camera prefix="camera1"/>
 	<joint name="${ns}camera_joint2" type="fixed">
-		<origin xyz="1.11 2.25 ${camera_offset_z}" rpy="0 0 0" />
+		<origin xyz="1.11 2.25 ${camera_offset_z}" rpy="0 0 0.7854" />
 		<parent link="${ns}base_link"/>
 		<child link="${ns}camera2_link"/>
@@ -20,5 +20,5 @@
 	<xacro:usb_camera prefix="camera2"/>
 	<joint name="${ns}camera_joint3" type="fixed">
-		<origin xyz="0 3.45 ${camera_offset_z}" rpy="0 0 0" />
+		<origin xyz="0 3.45 ${camera_offset_z}" rpy="0 0 1.5708" />
 		<parent link="${ns}base_link"/>
 		<child link="${ns}camera3_link"/>
@@ -26,5 +26,5 @@
 	<xacro:usb_camera prefix="camera3"/>
 	<joint name="${ns}camera_joint4" type="fixed">
-		<origin xyz="-1.11 2.25 ${camera_offset_z}" rpy="0 0 0" />
+		<origin xyz="-1.11 2.25 ${camera_offset_z}" rpy="0 0 2.3562" />
 		<parent link="${ns}base_link"/>
 		<child link="${ns}camera4_link"/>
@@ -32,5 +32,5 @@
 	<xacro:usb_camera prefix="camera4"/>
 	<joint name="${ns}camera_joint5" type="fixed">
-		<origin xyz="-1.82 0 ${camera_offset_z}" rpy="0 0 0" />
+		<origin xyz="-1.82 0 ${camera_offset_z}" rpy="0 0 3.1416" />
 		<parent link="${ns}base_link"/>
 		<child link="${ns}camera5_link"/>
@@ -38,5 +38,5 @@
 	<xacro:usb_camera prefix="camera5"/>
 	<joint name="${ns}camera_joint6" type="fixed">
-		<origin xyz="-1.31 -2.4375 ${camera_offset_z}" rpy="0 0 0" />
+		<origin xyz="-1.31 -2.4375 ${camera_offset_z}" rpy="0 0 3.9267" />
 		<parent link="${ns}base_link"/>
 		<child link="${ns}camera6_link"/>
@@ -44,5 +44,5 @@
 	<xacro:usb_camera prefix="camera6"/>
 	<joint name="${ns}camera_joint7" type="fixed">
-		<origin xyz="0 -3.825 ${camera_offset_z}" rpy="0 0 0" />
+		<origin xyz="0 -3.825 ${camera_offset_z}" rpy="0 0 4.7124" />
 		<parent link="${ns}base_link"/>
 		<child link="${ns}camera7_link"/>
@@ -50,5 +50,5 @@
 	<xacro:usb_camera prefix="camera7"/>
 	<joint name="${ns}camera_joint8" type="fixed">
-		<origin xyz="1.31 -2.4375 ${camera_offset_z}" rpy="0 0 0" />
+		<origin xyz="1.31 -2.4375 ${camera_offset_z}" rpy="0 0 5.4978" />
 		<parent link="${ns}base_link"/>
 		<child link="${ns}camera8_link"/>

File: cam/urdf/gazebo_robot.xacro (robot description, xacro)
@@ -151,5 +151,5 @@
                 <origin xyz=" 0 0 0" rpy="0 0 0" />
                 <geometry>
-                    <box size="4 8 0.1" />
+                    <box size="0.4 0.8 0.1" />
                 </geometry>
                 <material name="Yellow" />
